Commit message: collda files are added as replacement for too big fbx files

File: kitchenClash0.urdf (robot description, URDF)
Before this commit: robot KitchenClash0.urdf, 349 links, 348 joints
Links:
- link Cube: geometry visual mesh filename=package://h_neem/meshes/Cube.dae
- link Cube_1: geometry visual mesh filename=package://h_neem/meshes/Cube.dae
- link Cube_10: geometry visual mesh filename=package://h_neem/meshes/Cube.dae
- link Cube_11: geometry visual mesh filename=package://h_neem/meshes/Cube.dae
- link Cube_12: geometry visual mesh filename=package://h_neem/meshes/Cube.dae
- link Cube_13: geometry visual mesh filename=package://h_neem/meshes/Cube.dae
- link Cube_17042: geometry visual mesh filename=package://h_neem/meshes/Cube.dae
- link Cube_1_12959: geometry visual mesh filename=package://h_neem/meshes/Cube.dae
- link Cube_1_33376: geometry visual mesh filename=package://h_neem/meshes/Cube.dae
- link Cube_1_33534: geometry visual mesh filename=package://h_neem/meshes/Cube.dae
- link Cube_1_66524: geometry visual mesh filename=package://h_neem/meshes/Cube.dae
- link Cube_1_70777: geometry visual mesh filename=package://h_neem/meshes/Cube.dae
- link Cube_1_86271: geometry visual mesh filename=package://h_neem/meshes/Cube.dae
- link Cube_1_87286: geometry visual mesh filename=package://h_neem/meshes/Cube.dae
- link Cube_2: geometry visual mesh filename=package://h_neem/meshes/Cube.dae
- link Cube_21715: geometry visual mesh filename=package://h_neem/meshes/Cube.dae
- link Cube_21977: geometry visual mesh filename=package://h_neem/meshes/Cube.dae
- link Cube_2_31866: geometry visual mesh filename=package://h_neem/meshes/Cube.dae
- link Cube_2_60947: geometry visual mesh filename=package://h_neem/meshes/Cube.dae
- link Cube_2_61029: geometry visual mesh filename=package://h_neem/meshes/Cube.dae
- link Cube_2_70115: geometry visual mesh filename=package://h_neem/meshes/Cube.dae
- link Cube_2_70553: geometry visual mesh filename=package://h_neem/meshes/Cube.dae
- link Cube_2_8193: geometry visual mesh filename=package://h_neem/meshes/Cube.dae
- link Cube_2_99358: geometry visual mesh filename=package://h_neem/meshes/Cube.dae
- link Cube_3: geometry visual mesh filename=package://h_neem/meshes/Cube.dae
- link Cube_33884: geometry visual mesh filename=package://h_neem/meshes/Cube.dae
- link Cube_34343: geometry visual mesh filename=package://h_neem/meshes/Cube.dae
- link Cube_34559: geometry visual mesh filename=package://h_neem/meshes/Cube.dae
- link Cube_3736: geometry visual mesh filename=package://h_neem/meshes/Cube.dae
- link Cube_3_28928: geometry visual mesh filename=package://h_neem/meshes/Cube.dae
- link Cube_3_59990: geometry visual mesh filename=package://h_neem/meshes/Cube.dae
- link Cube_3_62137: geometry visual mesh filename=package://h_neem/meshes/Cube.dae
- link Cube_3_73054: geometry visual mesh filename=package://h_neem/meshes/Cube.dae
- link Cube_3_76169: geometry visual mesh filename=package://h_neem/meshes/Cube.dae
- link Cube_3_83299: geometry visual mesh filename=package://h_neem/meshes/Cube.dae
- link Cube_3_92970: geometry visual mesh filename=package://h_neem/meshes/Cube.dae
- link Cube_4: geometry visual mesh filename=package://h_neem/meshes/Cube.dae
- link Cube_44086: geometry visual mesh filename=package://h_neem/meshes/Cube.dae
- link Cube_4_14793: geometry visual mesh filename=package://h_neem/meshes/Cube.dae
- link Cube_4_49644: geometry visual mesh filename=package://h_neem/meshes/Cube.dae
- link Cube_4_56488: geometry visual mesh filename=package://h_neem/meshes/Cube.dae
- link Cube_4_65253: geometry visual mesh filename=package://h_neem/meshes/Cube.dae
- link Cube_5: geometry visual mesh filename=package://h_neem/meshes/Cube.dae
- link Cube_59574: geometry visual mesh filename=package://h_neem/meshes/Cube.dae
- link Cube_5_74574: geometry visual mesh filename=package://h_neem/meshes/Cube.dae
- link Cube_5_89013: geometry visual mesh filename=package://h_neem/meshes/Cube.dae
- link Cube_6: geometry visual mesh filename=package://h_neem/meshes/Cube.dae
- link Cube_60132: geometry visual mesh filename=package://h_neem/meshes/Cube.dae
- link Cube_62369: geometry visual mesh filename=package://h_neem/meshes/Cube.dae
- link Cube_68380: geometry visual mesh filename=package://h_neem/meshes/Cube.dae
- link Cube_6_41405: geometry visual mesh filename=package://h_neem/meshes/Cube.dae
- link Cube_6_77647: geometry visual mesh filename=package://h_neem/meshes/Cube.dae
- link Cube_7: geometry visual mesh filename=package://h_neem/meshes/Cube.dae
- link Cube_75106: geometry visual mesh filename=package://h_neem/meshes/Cube.dae
- link Cube_76983: geometry visual mesh filename=package://h_neem/meshes/Cube.dae
- link Cube_7_63222: geometry visual mesh filename=package://h_neem/meshes/Cube.dae
- link Cube_7_79703: geometry visual mesh filename=package://h_neem/meshes/Cube.dae
- link Cube_8: geometry visual mesh filename=package://h_neem/meshes/Cube.dae
- link Cube_81478: geometry visual mesh filename=package://h_neem/meshes/Cube.dae
- link Cube_84650: geometry visual mesh filename=package://h_neem/meshes/Cube.dae
- link Cube_87951: geometry visual mesh filename=package://h_neem/meshes/Cube.dae
- link Cube_9: geometry visual mesh filename=package://h_neem/meshes/Cube.dae
- link Cube_97832: geometry visual mesh filename=package://h_neem/meshes/Cube.dae
- link SO_RubixCube: geometry visual mesh filename=package://h_neem/meshes/Cube.dae
- link appleGreen: geometry visual mesh filename=package://h_neem/meshes/appleGreen.dae
- link appleGreen_1: geometry visual mesh filename=package://h_neem/meshes/appleGreen.dae
- link appleRed: geometry visual mesh filename=package://h_neem/meshes/appleRed.dae
- link apricot: geometry visual mesh filename=package://h_neem/meshes/apricot.dae
- link banana: geometry visual mesh filename=package://h_neem/meshes/banana.dae
- link bellPepperOrange: geometry visual mesh filename=package://h_neem/meshes/bellPepperOrange.dae
- link bellPepperYellow: geometry visual mesh filename=package://h_neem/meshes/bellPepperOrange.dae
- link bellpepperRed: geometry visual mesh filename=package://h_neem/meshes/bellPepperOrange.dae
- link broccoli: geometry visual mesh filename=package://h_neem/meshes/broccoli.dae
- link carrot: geometry visual mesh filename=package://h_neem/meshes/carrot.dae
- link cauliflower: geometry visual mesh filename=package://h_neem/meshes/cauliflower.dae
- link cherryRed: geometry visual mesh filename=package://h_neem/meshes/cherry.dae
- link chiliPepper: geometry visual mesh filename=package://h_neem/meshes/chiliPepper.dae
- link cucumber: geometry visual mesh filename=package://h_neem/meshes/cucumber.dae
- link eggplant: geometry visual mesh filename=package://h_neem/meshes/eggplant.dae
- link fig: geometry visual mesh filename=package://h_neem/meshes/fig.dae
- link garlic: geometry visual mesh filename=package://h_neem/meshes/garlic.dae
- link ground: geometry visual mesh filename=package://h_neem/meshes/Cube.dae
- link lemon: geometry visual mesh filename=package://h_neem/meshes/lemon.dae
- link lettuce: geometry visual mesh filename=package://h_neem/meshes/lettuce.dae
- link pawpaw: geometry visual mesh filename=package://h_neem/meshes/pawpaw.dae
- link potatoYellow: geometry visual mesh filename=package://h_neem/meshes/potatoBrown.dae
- link potatoYellow_1: geometry visual mesh filename=package://h_neem/meshes/potatoBrown.dae
- link radish: geometry visual mesh filename=package://h_neem/meshes/radish.dae
- link radish_1: geometry visual mesh filename=package://h_neem/meshes/radish.dae
- link radish_2: geometry visual mesh filename=package://h_neem/meshes/radish.dae
- link tomato: geometry visual mesh filename=package://h_neem/meshes/tomato.dae
