Commit message: collada meshes are used instead fbx

File: kitchenClash0.urdf (robot description, URDF)
Before this commit: robot KitchenClash0.urdf, 349 links, 348 joints
Links:
- removed link Öl
- added link Oil; visual mesh filename=package://h_neem/meshes/collada/Bottle4.dae
- link BathSink: geometry visual mesh filename=package://h_neem/meshes/collada/BathSink.dae
- link Bathtub: geometry visual mesh filename=package://h_neem/meshes/collada/Bathtub.dae
- link Bed: geometry visual mesh filename=package://h_neem/meshes/collada/Bed.dae
- link BigDrawer: geometry visual mesh filename=package://h_neem/meshes/collada/BigDrawer.dae
- link Book.1: geometry visual mesh filename=package://h_neem/meshes/collada/Book.1.dae
- link Book.2: geometry visual mesh filename=package://h_neem/meshes/collada/Book.2.dae
- link Book.3: geometry visual mesh filename=package://h_neem/meshes/collada/Book.3.dae
- link Book.4: geometry visual mesh filename=package://h_neem/meshes/collada/Book.4.dae
- link Book.5: geometry visual mesh filename=package://h_neem/meshes/collada/Book.4.dae
- link Bookshelf: geometry visual mesh filename=package://h_neem/meshes/collada/Bookshelf.dae
- link Bookshelf_1: geometry visual mesh filename=package://h_neem/meshes/collada/Bookshelf.dae
- link Bookshelf_2: geometry visual mesh filename=package://h_neem/meshes/collada/Bookshelf.dae
- link BoxshelfModel: geometry visual mesh filename=package://h_neem/meshes/collada/Boxshelf.dae
- link BroomBottom: geometry visual mesh filename=package://h_neem/meshes/collada/BroomBottom.dae
- link BroomTop: geometry visual mesh filename=package://h_neem/meshes/collada/BroomTop.dae
- link Chair: geometry visual mesh filename=package://h_neem/meshes/collada/Chair.dae
- link Chair_1: geometry visual mesh filename=package://h_neem/meshes/collada/Chair.dae
- link Chair_2: geometry visual mesh filename=package://h_neem/meshes/collada/Chair.dae
- link Chair_3: geometry visual mesh filename=package://h_neem/meshes/collada/Chair.dae
- link Cube: geometry visual mesh filename=package://h_neem/meshes/collada/Cube.dae
- link Cube_1: geometry visual mesh filename=package://h_neem/meshes/collada/Cube.dae
- link Cube_10: geometry visual mesh filename=package://h_neem/meshes/collada/Cube.dae
- link Cube_11: geometry visual mesh filename=package://h_neem/meshes/collada/Cube.dae
- link Cube_12: geometry visual mesh filename=package://h_neem/meshes/collada/Cube.dae
- link Cube_13: geometry visual mesh filename=package://h_neem/meshes/collada/Cube.dae
- link Cube_17042: geometry visual mesh filename=package://h_neem/meshes/collada/Cube.dae
- link Cube_1_12959: geometry visual mesh filename=package://h_neem/meshes/collada/Cube.dae
- link Cube_1_33376: geometry visual mesh filename=package://h_neem/meshes/collada/Cube.dae
- link Cube_1_33534: geometry visual mesh filename=package://h_neem/meshes/collada/Cube.dae
- link Cube_1_66524: geometry visual mesh filename=package://h_neem/meshes/collada/Cube.dae
- link Cube_1_70777: geometry visual mesh filename=package://h_neem/meshes/collada/Cube.dae
- link Cube_1_86271: geometry visual mesh filename=package://h_neem/meshes/collada/Cube.dae
- link Cube_1_87286: geometry visual mesh filename=package://h_neem/meshes/collada/Cube.dae
- link Cube_2: geometry visual mesh filename=package://h_neem/meshes/collada/Cube.dae
- link Cube_21715: geometry visual mesh filename=package://h_neem/meshes/collada/Cube.dae
- link Cube_21977: geometry visual mesh filename=package://h_neem/meshes/collada/Cube.dae
- link Cube_2_31866: geometry visual mesh filename=package://h_neem/meshes/collada/Cube.dae
- link Cube_2_60947: geometry visual mesh filename=package://h_neem/meshes/collada/Cube.dae
- link Cube_2_61029: geometry visual mesh filename=package://h_neem/meshes/collada/Cube.dae
- link Cube_2_70115: geometry visual mesh filename=package://h_neem/meshes/collada/Cube.dae
- link Cube_2_70553: geometry visual mesh filename=package://h_neem/meshes/collada/Cube.dae
- link Cube_2_8193: geometry visual mesh filename=package://h_neem/meshes/collada/Cube.dae
- link Cube_2_99358: geometry visual mesh filename=package://h_neem/meshes/collada/Cube.dae
- link Cube_3: geometry visual mesh filename=package://h_neem/meshes/collada/Cube.dae
- link Cube_33884: geometry visual mesh filename=package://h_neem/meshes/collada/Cube.dae
- link Cube_34343: geometry visual mesh filename=package://h_neem/meshes/collada/Cube.dae
- link Cube_34559: geometry visual mesh filename=package://h_neem/meshes/collada/Cube.dae
- link Cube_3736: geometry visual mesh filename=package://h_neem/meshes/collada/Cube.dae
- link Cube_3_28928: geometry visual mesh filename=package://h_neem/meshes/collada/Cube.dae
- link Cube_3_59990: geometry visual mesh filename=package://h_neem/meshes/collada/Cube.dae
- link Cube_3_62137: geometry visual mesh filename=package://h_neem/meshes/collada/Cube.dae
- link Cube_3_73054: geometry visual mesh filename=package://h_neem/meshes/collada/Cube.dae
- link Cube_3_76169: geometry visual mesh filename=package://h_neem/meshes/collada/Cube.dae
- link Cube_3_83299: geometry visual mesh filename=package://h_neem/meshes/collada/Cube.dae
- link Cube_3_92970: geometry visual mesh filename=package://h_neem/meshes/collada/Cube.dae
- link Cube_4: geometry visual mesh filename=package://h_neem/meshes/collada/Cube.dae
- link Cube_44086: geometry visual mesh filename=package://h_neem/meshes/collada/Cube.dae
- link Cube_4_14793: geometry visual mesh filename=package://h_neem/meshes/collada/Cube.dae
- link Cube_4_49644: geometry visual mesh filename=package://h_neem/meshes/collada/Cube.dae
- link Cube_4_56488: geometry visual mesh filename=package://h_neem/meshes/collada/Cube.dae
- link Cube_4_65253: geometry visual mesh filename=package://h_neem/meshes/collada/Cube.dae
- link Cube_5: geometry visual mesh filename=package://h_neem/meshes/collada/Cube.dae
- link Cube_59574: geometry visual mesh filename=package://h_neem/meshes/collada/Cube.dae
- link Cube_5_74574: geometry visual mesh filename=package://h_neem/meshes/collada/Cube.dae
- link Cube_5_89013: geometry visual mesh filename=package://h_neem/meshes/collada/Cube.dae
- link Cube_6: geometry visual mesh filename=package://h_neem/meshes/collada/Cube.dae
- link Cube_60132: geometry visual mesh filename=package://h_neem/meshes/collada/Cube.dae
- link Cube_62369: geometry visual mesh filename=package://h_neem/meshes/collada/Cube.dae
- link Cube_68380: geometry visual mesh filename=package://h_neem/meshes/collada/Cube.dae
- link Cube_6_41405: geometry visual mesh filename=package://h_neem/meshes/collada/Cube.dae
- link Cube_6_77647: geometry visual mesh filename=package://h_neem/meshes/collada/Cube.dae
- link Cube_7: geometry visual mesh filename=package://h_neem/meshes/collada/Cube.dae
- link Cube_75106: geometry visual mesh filename=package://h_neem/meshes/collada/Cube.dae
- link Cube_76983: geometry visual mesh filename=package://h_neem/meshes/collada/Cube.dae
- link Cube_7_63222: geometry visual mesh filename=package://h_neem/meshes/collada/Cube.dae
- link Cube_7_79703: geometry visual mesh filename=package://h_neem/meshes/collada/Cube.dae
- link Cube_8: geometry visual mesh filename=package://h_neem/meshes/collada/Cube.dae
- link Cube_81478: geometry visual mesh filename=package://h_neem/meshes/collada/Cube.dae
- link Cube_84650: geometry visual mesh filename=package://h_neem/meshes/collada/Cube.dae
- link Cube_87951: geometry visual mesh filename=package://h_neem/meshes/collada/Cube.dae
- link Cube_9: geometry visual mesh filename=package://h_neem/meshes/collada/Cube.dae
- link Cube_97832: geometry visual mesh filename=package://h_neem/meshes/collada/Cube.dae
- link Door_02: geometry visual mesh filename=package://h_neem/meshes/collada/Door.dae
- link Door_02_1: geometry visual mesh filename=package://h_neem/meshes/collada/Door.dae
- link Drawer: geometry visual mesh filename=package://h_neem/meshes/collada/Drawer.dae
- link Drawer_1: geometry visual mesh filename=package://h_neem/meshes/collada/Drawer.dae
- link Drawer_2: geometry visual mesh filename=package://h_neem/meshes/collada/Drawer.dae
- link Floor_Carpet_Grey: geometry visual mesh filename=package://h_neem/meshes/collada/Floor_Carpet_Grey.dae
- link Floor_Carpet_Tiles: geometry visual mesh filename=package://h_neem/meshes/collada/Floor_Carpet_Tiles.dae
- link Floor_Carpet_Tiles_1: geometry visual mesh filename=package://h_neem/meshes/collada/Floor_Carpet_Tiles.dae
- link Floor_Carpet_Tiles_2: geometry visual mesh filename=package://h_neem/meshes/collada/Floor_Carpet_Tiles.dae
- link Floor_Carpet_Tiles_3: geometry visual mesh filename=package://h_neem/meshes/collada/Floor_Carpet_Tiles.dae
- link Floor_Carpet_Tiles_4: geometry visual mesh filename=package://h_neem/meshes/collada/Floor_Carpet_Tiles.dae
- link Floor_Carpet_Tiles_5: geometry visual mesh filename=package://h_neem/meshes/collada/Floor_Carpet_Tiles.dae
- link Floor_Carpet_Tiles_6: geometry visual mesh filename=package://h_neem/meshes/collada/Floor_Carpet_Tiles.dae
- link Floor_Carpet_Tiles_7: geometry visual mesh filename=package://h_neem/meshes/collada/Floor_Carpet_Tiles.dae
- link Floor_Carpet_Tiles_8: geometry visual mesh filename=package://h_neem/meshes/collada/Floor_Carpet_Tiles.dae
- link Floor_Vinyl: geometry visual mesh filename=package://h_neem/meshes/collada/Floor_Vinyl.dae
- link Floor_Wood: geometry visual mesh filename=package://h_neem/meshes/collada/Floor_Wood.dae
- link Floor_Wood_1: geometry visual mesh filename=package://h_neem/meshes/collada/Floor_Wood.dae
- link Floor_Wood_10: geometry visual mesh filename=package://h_neem/meshes/collada/Floor_Wood.dae
- link Floor_Wood_11: geometry visual mesh filename=package://h_neem/meshes/collada/Floor_Wood.dae
- link Floor_Wood_2: geometry visual mesh filename=package://h_neem/meshes/collada/Floor_Wood.dae
- link Floor_Wood_3: geometry visual mesh filename=package://h_neem/meshes/collada/Floor_Wood.dae
- link Floor_Wood_4: geometry visual mesh filename=package://h_neem/meshes/collada/Floor_Wood.dae
- link Floor_Wood_5: geometry visual mesh filename=package://h_neem/meshes/collada/Floor_Wood.dae
- link Floor_Wood_6: geometry visual mesh filename=package://h_neem/meshes/collada/Floor_Wood.dae
- link Floor_Wood_7: geometry visual mesh filename=package://h_neem/meshes/collada/Floor_Wood.dae
- link Floor_Wood_8: geometry visual mesh filename=package://h_neem/meshes/collada/Floor_Wood.dae
- link Floor_Wood_9: geometry visual mesh filename=package://h_neem/meshes/collada/Floor_Wood.dae
- link Items_CrowBar_01: geometry visual mesh filename=package://h_neem/meshes/collada/Items_CrowBar_01.dae
- link Items_Drill_01: geometry visual mesh filename=package://h_neem/meshes/collada/Items_Drill_01.dae
- link Items_FlashLight_01: geometry visual mesh filename=package://h_neem/meshes/collada/Items_FlashLight_01.dae
- link Items_FryPan_01: geometry visual mesh filename=package://h_neem/meshes/collada/Items_FryPan_01.dae
- link Items_Hammer_01: geometry visual mesh filename=package://h_neem/meshes/collada/Items_Hammer_01.dae
- link Items_ScrewDriver_01: geometry visual mesh filename=package://h_neem/meshes/collada/Items_ScrewDriver_01.dae
- link Items_ScrewDriver_02: geometry visual mesh filename=package://h_neem/meshes/collada/Items_ScrewDriver_02.dae
- link Items_ScrewDriver_03: geometry visual mesh filename=package://h_neem/meshes/collada/Items_ScrewDriver_03.dae
- link Items_SledgeHammer_01: geometry visual mesh filename=package://h_neem/meshes/collada/Items_SledgeHammer_01.dae
- link Items_SmartPhone_01: geometry visual mesh filename=package://h_neem/meshes/collada/Items_SmartPhone_01.dae
- link Items_Spanner_01: geometry visual mesh filename=package://h_neem/meshes/collada/Items_Spanner_01.dae
- link Items_Wrench_01: geometry visual mesh filename=package://h_neem/meshes/collada/Items_Wrench_01.dae
- link Lamp: geometry visual mesh filename=package://h_neem/meshes/collada/Lamp.dae
- link MicrowaveBack: geometry visual mesh filename=package://h_neem/meshes/collada/MicrowaveBack.dae
- link MicrowaveFrontModel: geometry visual mesh filename=package://h_neem/meshes/collada/MicrowaveFront.dae
- link Mirror: geometry visual mesh filename=package://h_neem/meshes/collada/Mirror.dae
- link Mirror.1: geometry visual mesh filename=package://h_neem/meshes/collada/Mirror.1.dae
- link Plunger: geometry visual mesh filename=package://h_neem/meshes/collada/Plunger.dae
- link Prop_Bar_Bench: geometry visual mesh filename=package://h_neem/meshes/collada/Prop_Bar_Bench.dae
- link Prop_BathMat_Blue: geometry visual mesh filename=package://h_neem/meshes/collada/Prop_BathMat_Blue.dae
- link Prop_Big_Clock: geometry visual mesh filename=package://h_neem/meshes/collada/Prop_Big_Clock.dae
- link Prop_Bonzai: geometry visual mesh filename=package://h_neem/meshes/collada/Prop_Bonzai.dae
- link Prop_Cupboard_03: geometry visual mesh filename=package://h_neem/meshes/collada/Prop_Cupboard_03.dae
- link Prop_Curtains_Blue: geometry visual mesh filename=package://h_neem/meshes/collada/Prop_Curtains_Blue.dae
- link Prop_Curtains_Blue_1: geometry visual mesh filename=package://h_neem/meshes/collada/Prop_Curtains_Blue.dae
- link Prop_Curtains_Blue_2: geometry visual mesh filename=package://h_neem/meshes/collada/Prop_Curtains_Blue.dae
- link Prop_Curtains_Blue_3: geometry visual mesh filename=package://h_neem/meshes/collada/Prop_Curtains_Blue.dae
- link Prop_Curtains_Red: geometry visual mesh filename=package://h_neem/meshes/collada/Prop_Curtains_Red.dae
- link Prop_Curtains_Red_1: geometry visual mesh filename=package://h_neem/meshes/collada/Prop_Curtains_Red.dae
- link Prop_Fireplace_02: geometry visual mesh filename=package://h_neem/meshes/collada/Prop_Fireplace_02.dae
- link Prop_Plant: geometry visual mesh filename=package://h_neem/meshes/collada/Prop_Plant.dae
- link Prop_Plant_02: geometry visual mesh filename=package://h_neem/meshes/collada/Prop_Plant.dae
- link Prop_Rug_03: geometry visual mesh filename=package://h_neem/meshes/collada/Prop_Rug_03.dae
- link Prop_Shelf_011: geometry visual mesh filename=package://h_neem/meshes/collada/Prop_Shelf_011.dae
- link Prop_Shelf_011_2: geometry visual mesh filename=package://h_neem/meshes/collada/Prop_Shelf_011.dae
- link Prop_Shelf_04: geometry visual mesh filename=package://h_neem/meshes/collada/Prop_Shelf_04.dae
- link Prop_Speaker_02: geometry visual mesh filename=package://h_neem/meshes/collada/pea.dae
- link Prop_Speaker_02_1: geometry visual mesh filename=package://h_neem/meshes/collada/pea.dae
- link Prop_ToiletSeat_01: geometry visual mesh filename=package://h_neem/meshes/collada/Prop_ToiletSeat_01.dae
- link Prop_Toilet_01: geometry visual mesh filename=package://h_neem/meshes/collada/Prop_Toilet_01.dae
- link Prop_WallArt_01: geometry visual mesh filename=package://h_neem/meshes/collada/Prop_WallArt_01.dae
- link Prop_WallArt_02: geometry visual mesh filename=package://h_neem/meshes/collada/Prop_WallArt_02.dae
- link Prop_WallArt_03: geometry visual mesh filename=package://h_neem/meshes/collada/Prop_WallArt_03.dae
- link Prop_shelf_01: geometry visual mesh filename=package://h_neem/meshes/collada/Prop_shelf_01.dae
- link Prop_shelf_01_1: geometry visual mesh filename=package://h_neem/meshes/collada/Prop_shelf_01.dae
- link Refridgerator_Door: geometry visual mesh filename=package://h_neem/meshes/collada/Refridgerator_Door.dae
- link Refridgerator_Empty: geometry visual mesh filename=package://h_neem/meshes/collada/Refridgerator_Empty.dae
- link Refridgerator_UpperDrawer: geometry visual mesh filename=package://h_neem/meshes/collada/Refridgerator_UpperDrawer.d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
- link SI_Env_Wall_01: geometry visual mesh filename=package://h_neem/meshes/collada/SI_Env_Wall_01.dae
- link SI_Env_Wall_01_1: geometry visual mesh filename=package://h_neem/meshes/collada/SI_Env_Wall_01.dae
- link SI_Env_Wall_01_10: geometry visual mesh filename=package://h_neem/meshes/collada/SI_Env_Wall_01.dae
- link SI_Env_Wall_01_11: geometry visual mesh filename=package://h_neem/meshes/collada/SI_Env_Wall_01.dae
- link SI_Env_Wall_01_12: geometry visual mesh filename=package://h_neem/meshes/collada/SI_Env_Wall_01.dae
- link SI_Env_Wall_01_13: geometry visual mesh filename=package://h_neem/meshes/collada/SI_Env_Wall_01.dae
- link SI_Env_Wall_01_14: geometry visual mesh filename=package://h_neem/meshes/collada/SI_Env_Wall_01.dae
- link SI_Env_Wall_01_15: geometry visual mesh filename=package://h_neem/meshes/collada/SI_Env_Wall_01.dae
- link SI_Env_Wall_01_16: geometry visual mesh filename=package://h_neem/meshes/collada/SI_Env_Wall_01.dae
- link SI_Env_Wall_01_17: geometry visual mesh filename=package://h_neem/meshes/collada/SI_Env_Wall_01.dae
- link SI_Env_Wall_01_18: geometry visual mesh filename=package://h_neem/meshes/collada/SI_Env_Wall_01.dae
- link SI_Env_Wall_01_19: geometry visual mesh filename=package://h_neem/meshes/collada/SI_Env_Wall_01.dae
- link SI_Env_Wall_01_2: geometry visual mesh filename=package://h_neem/meshes/collada/SI_Env_Wall_01.dae
- link SI_Env_Wall_01_20: geometry visual mesh filename=package://h_neem/meshes/collada/SI_Env_Wall_01.dae
- link SI_Env_Wall_01_21: geometry visual mesh filename=package://h_neem/meshes/collada/SI_Env_Wall_01.dae
- link SI_Env_Wall_01_22: geometry visual mesh filename=package://h_neem/meshes/collada/SI_Env_Wall_01.dae
- link SI_Env_Wall_01_23: geometry visual mesh filename=package://h_neem/meshes/collada/SI_Env_Wall_01.dae
- link SI_Env_Wall_01_24: geometry visual mesh filename=package://h_neem/meshes/collada/SI_Env_Wall_01.dae
- link SI_Env_Wall_01_25: geometry visual mesh filename=package://h_neem/meshes/collada/SI_Env_Wall_01.dae
- link SI_Env_Wall_01_26: geometry visual mesh filename=package://h_neem/meshes/collada/SI_Env_Wall_01.dae
- link SI_Env_Wall_01_27: geometry visual mesh filename=package://h_neem/meshes/collada/SI_Env_Wall_01.dae
- link SI_Env_Wall_01_28: geometry visual mesh filename=package://h_neem/meshes/collada/SI_Env_Wall_01.dae
- link SI_Env_Wall_01_29: geometry visual mesh filename=package://h_neem/meshes/collada/SI_Env_Wall_01.dae
- link SI_Env_Wall_01_3: geometry visual mesh filename=package://h_neem/meshes/collada/SI_Env_Wall_01.dae
- link SI_Env_Wall_01_30: geometry visual mesh filename=package://h_neem/meshes/collada/SI_Env_Wall_01.dae
- link SI_Env_Wall_01_31: geometry visual mesh filename=package://h_neem/meshes/collada/SI_Env_Wall_01.dae
- link SI_Env_Wall_01_32: geometry visual mesh filename=package://h_neem/meshes/collada/SI_Env_Wall_01.dae
- link SI_Env_Wall_01_33: geometry visual mesh filename=package://h_neem/meshes/collada/SI_Env_Wall_01.dae
- link SI_Env_Wall_01_34: geometry visual mesh filename=package://h_neem/meshes/collada/SI_Env_Wall_01.dae
- link SI_Env_Wall_01_35: geometry visual mesh filename=package://h_neem/meshes/collada/SI_Env_Wall_01.dae
- link SI_Env_Wall_01_4: geometry visual mesh filename=package://h_neem/meshes/collada/SI_Env_Wall_01.dae
- link SI_Env_Wall_01_5: geometry visual mesh filename=package://h_neem/meshes/collada/SI_Env_Wall_01.dae
- link SI_Env_Wall_01_6: geometry visual mesh filename=package://h_neem/meshes/collada/SI_Env_Wall_01.dae
- link SI_Env_Wall_01_7: geometry visual mesh filename=package://h_neem/meshes/collada/SI_Env_Wall_01.dae
- link SI_Env_Wall_01_8: geometry visual mesh filename=package://h_neem/meshes/collada/SI_Env_Wall_01.dae
- link SI_Env_Wall_01_9: geometry visual mesh filename=package://h_neem/meshes/collada/SI_Env_Wall_01.dae
- link SI_Env_Wall_CornerBlock_large: geometry visual mesh filename=package://h_neem/meshes/collada/SI_Env_Wall_CornerBlock.dae
- link SI_Env_Wall_CornerBlock_large_1: geometry visual mesh filename=package://h_neem/meshes/collada/SI_Env_Wall_CornerBlock.dae
- link SI_Env_Wall_CornerBlock_large_10: geometry visual mesh filename=package://h_neem/meshes/collada/SI_Env_Wall_CornerBlock.dae
- link SI_Env_Wall_CornerBlock_large_11: geometry visual mesh filename=package://h_neem/meshes/collada/SI_Env_Wall_CornerBlock.dae
- link SI_Env_Wall_CornerBlock_large_2: geometry visual mesh filename=package://h_neem/meshes/collada/SI_Env_Wall_CornerBlock.dae
- link SI_Env_Wall_CornerBlock_large_3: geometry visual mesh filename=package://h_neem/meshes/collada/SI_Env_Wall_CornerBlock.dae
- link SI_Env_Wall_CornerBlock_large_4: geometry visual mesh filename=package://h_neem/meshes/collada/SI_Env_Wall_CornerBlock.dae
- link SI_Env_Wall_CornerBlock_large_5: geometry visual mesh filename=package://h_neem/meshes/collada/SI_Env_Wall_CornerBlock.dae
- link SI_Env_Wall_CornerBlock_large_6: geometry visual mesh filename=package://h_neem/meshes/collada/SI_Env_Wall_CornerBlock.dae
- link SI_Env_Wall_CornerBlock_large_7: geometry visual mesh filename=package://h_neem/meshes/collada/SI_Env_Wall_CornerBlock.dae
- link SI_Env_Wall_CornerBlock_large_8: geometry visual mesh filename=package://h_neem/meshes/collada/SI_Env_Wall_CornerBlock.dae
- link SI_Env_Wall_CornerBlock_large_9: geometry visual mesh filename=package://h_neem/meshes/collada/SI_Env_Wall_CornerBlock.dae
- link SI_Env_Wall_Door_Small_01: geometry visual mesh filename=package://h_neem/meshes/collada/Door.dae
- link SI_Env_Wall_Door_Small_01_1: geometry visual mesh filename=package://h_neem/meshes/collada/Door.dae
- link SI_Env_Wall_Door_Small_01_2: geometry visual mesh filename=package://h_neem/meshes/collada/Door.dae
- link SI_Env_Wall_Large_Window_05: geometry visual mesh filename=package://h_neem/meshes/collada/SI_Env_Wall_Large_Window_05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
- link SI_Env_Wall_Large_Window_05_1: geometry visual mesh filename=package://h_neem/meshes/collada/SI_Env_Wall_Large_Window_05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
- link SI_Env_Wall_Large_Window_05_2: geometry visual mesh filename=package://h_neem/meshes/collada/SI_Env_Wall_Large_Window_05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
- link SI_Env_Wall_Large_Window_05_3: geometry visual mesh filename=package://h_neem/meshes/collada/SI_Env_Wall_Large_Window_05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
- link SI_Env_Wall_Large_Window_05_4: geometry visual mesh filename=package://h_neem/meshes/collada/SI_Env_Wall_Large_Window_05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
- link SI_Env_Wall_Large_Window_05_5: geometry visual mesh filename=package://h_neem/meshes/collada/SI_Env_Wall_Large_Window_05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
- link SI_Env_Wall_Large_Window_05_6: geometry visual mesh filename=package://h_neem/meshes/collada/SI_Env_Wall_Large_Window_05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
- link SI_Food_Meat_Steak_Raw: geometry visual mesh filename=package://h_neem/meshes/collada/SI_Food_Meat_Steak_Raw.dae
- link SM_Bowl: geometry visual mesh filename=package://h_neem/meshes/collada/Bowl.dae
- link SM_Bowl_1: geometry visual mesh filename=package://h_neem/meshes/collada/Bowl.dae
- link SM_Bowl_2: geometry visual mesh filename=package://h_neem/meshes/collada/Bowl.dae
- link SM_Bowl_3: geometry visual mesh filename=package://h_neem/meshes/collada/Bowl.dae
- link SM_Bowl_Small: geometry visual mesh filename=package://h_neem/meshes/collada/Bowl.dae
- link SM_Bowl_Small_1: geometry visual mesh filename=package://h_neem/meshes/collada/Bowl.dae
- link SM_Bowl_Small_2: geometry visual mesh filename=package://h_neem/meshes/collada/Bowl.dae
- link SM_Bowl_Small_3: geometry visual mesh filename=package://h_neem/meshes/collada/Bowl.dae
- link SM_Fork_Dinner: geometry visual mesh filename=package://h_neem/meshes/collada/SM_Fork_Dinner.dae
- link SM_Fork_Dinner_15572: geometry visual mesh filename=package://h_neem/meshes/collada/SM_Fork_Dinner.dae
- link SM_Fork_Dinner_17398: geometry visual mesh filename=package://h_neem/meshes/collada/SM_Fork_Dinner.dae
- link SM_Fork_Dinner_69885: geometry visual mesh filename=package://h_neem/meshes/collada/SM_Fork_Dinner.dae
- link SM_Knife_Table: geometry visual mesh filename=package://h_neem/meshes/collada/SM_Knife_Table.dae
- link SM_Knife_Table_12175: geometry visual mesh filename=package://h_neem/meshes/collada/SM_Knife_Table.dae
- link SM_Knife_Table_48929: geometry visual mesh filename=package://h_neem/meshes/collada/SM_Knife_Table.dae
- link SM_Knife_Table_84538: geometry visual mesh filename=package://h_neem/meshes/collada/SM_Knife_Table.dae
- link SM_Plate_Classic_16cm: geometry visual mesh filename=package://h_neem/meshes/collada/SM_Plate_Classic_16cm.dae
- link SM_Plate_Classic_16cm_1: geometry visual mesh filename=package://h_neem/meshes/collada/SM_Plate_Classic_16cm.dae
- link SM_Plate_Classic_16cm_2: geometry visual mesh filename=package://h_neem/meshes/collada/SM_Plate_Classic_16cm.dae
- link SM_Plate_Classic_16cm_3: geometry visual mesh filename=package://h_neem/meshes/collada/SM_Plate_Classic_16cm.dae
- link SM_Plate_Classic_21cm: geometry visual mesh filename=package://h_neem/meshes/collada/SM_Plate_Classic_21cm.dae
- link SM_Plate_Classic_21cm_1: geometry visual mesh filename=package://h_neem/meshes/collada/SM_Plate_Classic_21cm.dae
- link SM_Plate_Classic_21cm_2: geometry visual mesh filename=package://h_neem/meshes/collada/SM_Plate_Classic_21cm.dae
- link SM_Plate_Classic_21cm_3: geometry visual mesh filename=package://h_neem/meshes/collada/SM_Plate_Classic_21cm.dae
- link SM_Plate_Classic_26cm: geometry visual mesh filename=package://h_neem/meshes/collada/SM_Plate_Classic_26cm.dae
- link SM_Plate_Classic_26cm_1: geometry visual mesh filename=package://h_neem/meshes/collada/SM_Plate_Classic_26cm.dae
- link SM_Plate_Classic_26cm_2: geometry visual mesh filename=package://h_neem/meshes/collada/SM_Plate_Classic_26cm.dae
- link SM_Plate_Classic_26cm_3: geometry visual mesh filename=package://h_neem/meshes/collada/SM_Plate_Classic_26cm.dae
- link SM_Saucer: geometry visual mesh filename=package://h_neem/meshes/collada/SM_Saucer.dae
- link SM_Saucer_1: geometry visual mesh filename=package://h_neem/meshes/collada/SM_Saucer.dae
- link SM_Saucer_2: geometry visual mesh filename=package://h_neem/meshes/collada/SM_Saucer.dae
- link SM_Saucer_3: geometry visual mesh filename=package://h_neem/meshes/collada/SM_Saucer.dae
- link SM_Spoon_Soup: geometry visual mesh filename=package://h_neem/meshes/collada/SM_Spoon_Soup.dae
- link SM_Spoon_Soup_10143: geometry visual mesh filename=package://h_neem/meshes/collada/SM_Spoon_Soup.dae
- link SM_Spoon_Soup_24722: geometry visual mesh filename=package://h_neem/meshes/collada/SM_Spoon_Soup.dae
- link SM_Spoon_Soup_88278: geometry visual mesh filename=package://h_neem/meshes/collada/SM_Spoon_Soup.dae
- link SM_TraySet_Mid: geometry visual mesh filename=package://h_neem/meshes/collada/SM_TraySet_Mid.dae
- link SO_Boxfile_01: geometry visual mesh filename=package://h_neem/meshes/collada/SO_Boxfile_01.dae
- link SO_Boxfile_03: geometry visual mesh filename=package://h_neem/meshes/collada/SO_Boxfile_03.dae
- link SO_Boxfile_05: geometry visual mesh filename=package://h_neem/meshes/collada/SO_Boxfile_05.dae
- link SO_Boxfile_06: geometry visual mesh filename=package://h_neem/meshes/collada/SO_Boxfile_06.dae
- link SO_Broom: geometry visual mesh filename=package://h_neem/meshes/collada/Broom.dae
- link SO_CarboardBox_01: geometry visual mesh filename=package://h_neem/meshes/collada/SO_CarboardBox_01.dae
- link SO_Clipboard: geometry visual mesh filename=package://h_neem/meshes/collada/SO_Clipboard.dae
- link SO_Papers_03: geometry visual mesh filename=package://h_neem/meshes/collada/SO_Papers_03.dae
- link SO_Pen_01: geometry visual mesh filename=package://h_neem/meshes/collada/SO_Pen_01.dae
- link SO_Pen_02: geometry visual mesh filename=package://h_neem/meshes/collada/SO_Pen_02.dae
- link SO_Pinboard_01: geometry visual mesh filename=package://h_neem/meshes/collada/SO_Pinboard_01.dae
- link SO_Plant_01: geometry visual mesh filename=package://h_neem/meshes/collada/SO_Plant_01.dae
- link SO_Plant_02: geometry visual mesh filename=package://h_neem/meshes/collada/SO_Plant_02.dae
- link SO_Plant_03: geometry visual mesh filename=package://h_neem/meshes/collada/SO_Plant_03.dae
- link SO_RubixCube: geometry visual mesh filename=package://h_neem/meshes/collada/Cube.dae
- link SO_Rug_01: geometry visual mesh filename=package://h_neem/meshes/collada/SO_Rug_01.dae
- link Sink.2: geometry visual mesh filename=package://h_neem/meshes/collada/Sink.2.dae
- link Sink1_DoorL: geometry visual mesh filename=package://h_neem/meshes/collada/Sink1_DoorL.dae
- link Sink1_DoorR: geometry visual mesh filename=package://h_neem/meshes/collada/Sink1_DoorR.dae
- link Sink1_Drawer2: geometry visual mesh filename=package://h_neem/meshes/collada/Sink1_Drawer2.dae
- link Sink1_Drawer3: geometry visual mesh filename=package://h_neem/meshes/collada/Sink1_Drawer3.dae
- link Sink1_Drawer4: geometry visual mesh filename=package://h_neem/meshes/collada/Sink1_Drawer4.dae
- link Sink1_Drawer5: geometry visual mesh filename=package://h_neem/meshes/collada/Sink1_Drawer5.dae
- link Sink1_Empty: geometry visual mesh filename=package://h_neem/meshes/collada/Sink1_Empty.dae
- link Sink1_OvenDoor: geometry visual mesh filename=package://h_neem/meshes/collada/Sink1_OvenDoor.dae
- link Sink1_SinkDoor: geometry visual mesh filename=package://h_neem/meshes/collada/Sink1_SinkDoor.dae
- link Sink_DoorL: geometry visual mesh filename=package://h_neem/meshes/collada/Sink_DoorL.dae
- link Sink_DoorR: geometry visual mesh filename=package://h_neem/meshes/collada/Sink_DoorR.dae
- link Sink_Drawer1: geometry visual mesh filename=package://h_neem/meshes/collada/Sink_Drawer1.dae
- link Sink_Drawer2: geometry visual mesh filename=package://h_neem/meshes/collada/Sink_Drawer2.dae
- link Sink_WithoutDrawers: geometry visual mesh filename=package://h_neem/meshes/collada/Sink_WithoutDrawers.dae
- link Sofa.1: geometry visual mesh filename=package://h_neem/meshes/collada/Sofa.1.dae
- link TV: geometry visual mesh filename=package://h_neem/meshes/collada/TV.dae
- link TVTable: geometry visual mesh filename=package://h_neem/meshes/collada/TVTable.dae
- link Table: geometry visual mesh filename=package://h_neem/meshes/collada/Table.dae
- link TallLamp: geometry visual mesh filename=package://h_neem/meshes/collada/TallLamp.dae
- link Toilet_Paper: geometry visual mesh filename=package://h_neem/meshes/collada/Toilet.dae
- link Towel_Rack: geometry visual mesh filename=package://h_neem/meshes/collada/Towel_Rack.dae
- link Trashcan1: geometry visual mesh filename=package://h_neem/meshes/collada/Trash.dae
- link Trashcan1Cap: geometry visual mesh filename=package://h_neem/meshes/collada/Trash.dae
- link Upper: geometry visual mesh filename=package://h_neem/meshes/collada/Boxshelf.dae
- link Wall_01_Blue: geometry visual mesh filename=package://h_neem/meshes/collada/Wall_01_Blue.dae
- link Wall_01_Blue_1: geometry visual mesh filename=package://h_neem/meshes/collada/Wall_01_Blue.dae
- link Wall_01_Blue_2: geometry visual mesh filename=package://h_neem/meshes/collada/Wall_01_Blue.dae
- link Wall_01_Blue_3: geometry visual mesh filename=package://h_neem/meshes/collada/Wall_01_Blue.dae
- link Wall_01_Blue_4: geometry visual mesh filename=package://h_neem/meshes/collada/Wall_01_Blue.dae
- link Wall_01_Blue_5: geometry visual mesh filename=package://h_neem/meshes/collada/Wall_01_Blue.dae
- link Wall_01_Blue_6: geometry visual mesh filename=package://h_neem/meshes/collada/Wall_01_Blue.dae
- link Wall_01_Blue_7: geometry visual mesh filename=package://h_neem/meshes/collada/Wall_01_Blue.dae
- link Wall_01_Blue_8: geometry visual mesh filename=package://h_neem/meshes/collada/Wall_01_Blue.dae
- link Wall_Door_01_Blue_1: geometry visual mesh filename=package://h_neem/meshes/collada/Door.dae
- link Wall_Window_01_Blue: geometry visual mesh filename=package://h_neem/meshes/collada/Wall_Window_01_Blue.dae
- link appleGreen: geometry visual mesh filename=package://h_neem/meshes/collada/appleGreen.dae
- link appleGreen_1: geometry visual mesh filename=package://h_neem/meshes/collada/appleGreen.dae
- link appleRed: geometry visual mesh filename=package://h_neem/meshes/collada/appleRed.dae
- link apricot: geometry visual mesh filename=package://h_neem/meshes/collada/apricot.dae
- link banana: geometry visual mesh filename=package://h_neem/meshes/collada/banana.dae
- link bellPepperOrange: geometry visual mesh filename=package://h_neem/meshes/collada/bellPepperOrange.dae
- link bellPepperYellow: geometry visual mesh filename=package://h_neem/meshes/collada/bellPepperOrange.dae
- link bellpepperRed: geometry visual mesh filename=package://h_neem/meshes/collada/bellPepperOrange.dae
- link broccoli: geometry visual mesh filename=package://h_neem/meshes/collada/broccoli.dae
- link carrot: geometry visual mesh filename=package://h_neem/meshes/collada/carrot.dae
- link cauliflower: geometry visual mesh filename=package://h_neem/meshes/collada/cauliflower.dae
- link cherryRed: geometry visual mesh filename=package://h_neem/meshes/collada/cherry.dae
- link chiliPepper: geometry visual mesh filename=package://h_neem/meshes/collada/chiliPepper.dae
- link cucumber: geometry visual mesh filename=package://h_neem/meshes/collada/cucumber.dae
- link eggplant: geometry visual mesh filename=package://h_neem/meshes/collada/eggplant.dae
- link fig: geometry visual mesh filename=package://h_neem/meshes/collada/fig.dae
- link garlic: geometry visual mesh filename=package://h_neem/meshes/collada/garlic.dae
- link ground: geometry visual mesh filename=package://h_neem/meshes/collada/Cube.dae
- link lemon: geometry visual mesh filename=package://h_neem/meshes/collada/lemon.dae
- link lettuce: geometry visual mesh filename=package://h_neem/meshes/collada/lettuce.dae
- link pawpaw: geometry visual mesh filename=package://h_neem/meshes/collada/pawpaw.dae
- link potatoYellow: geometry visual mesh filename=package://h_neem/meshes/collada/potatoBrown.dae
- link potatoYellow_1: geometry visual mesh filename=package://h_neem/meshes/collada/potatoBrown.dae
- link radish: geometry visual mesh filename=package://h_neem/meshes/collada/radish.dae
- link radish_1: geometry visual mesh filename=package://h_neem/meshes/collada/radish.dae
- link radish_2: geometry visual mesh filename=package://h_neem/meshes/collada/radish.dae
- link scp_mw_axe: geometry visual mesh filename=package://h_neem/meshes/collada/scp_mw_axe.dae
- link scp_mw_baseball_bat_02: geometry visual mesh filename=package://h_neem/meshes/collada/scp_mw_baseball_bat_01.dae
- link scp_mw_cleaver_knife_02: geometry visual mesh filename=package://h_neem/meshes/collada/scp_mw_cleaver_knife_02.dae
- link scp_mw_fire_poker: geometry visual mesh filename=package://h_neem/meshes/collada/scp_mw_fire_poker.dae
- link scp_mw_flyswatter_01: geometry visual mesh filename=package://h_neem/meshes/collada/scp_mw_flyswatter_01.dae
- link scp_mw_flyswatter_02: geometry visual mesh filename=package://h_neem/meshes/collada/scp_mw_flyswatter_01.dae
- link scp_mw_kitchen_fork: geometry visual mesh filename=package://h_neem/meshes/collada/scp_mw_kitchen_fork.dae
- link scp_mw_kitchen_turner: geometry visual mesh filename=package://h_neem/meshes/collada/scp_mw_kitchen_turner.dae
- link scp_mw_knife_01: geometry visual mesh filename=package://h_neem/meshes/collada/scp_mw_knife_01.dae
- link scp_mw_knife_01_1: geometry visual mesh filename=package://h_neem/meshes/collada/scp_mw_knife_01.dae
- link scp_mw_knife_01_2: geometry visual mesh filename=package://h_neem/meshes/collada/scp_mw_knife_01.dae
- link scp_mw_knife_01_2_92314: geometry visual mesh filename=package://h_neem/meshes/collada/scp_mw_knife_01.dae
- link scp_mw_rolling_pin: geometry visual mesh filename=package://h_neem/meshes/collada/scp_mw_rolling_pin.dae
- link tomato: geometry visual mesh filename=package://h_neem/meshes/collada/tomato.dae
Joints:
- removed joint Öl_joint
- added joint oil_joint: type fixed, parent room_link, child Oil, origin xyz=-17.384 2.062249 -0.222 rpy=270 39.0218 0, axis 0 0 0, limit lower=0 upper=0 effort=300 velocity=10
