Commit message: status

File: kitchenClash0.urdf (robot description, URDF)
Before this commit: robot KitchenClash0.urdf, 349 links, 348 joints
Joints:
- joint BathSink_joint: origin xyz=13.4 1.02 10.81 rpy=0 180 0 -> (none)
- joint Bathtub_joint: origin xyz=17.97 -0.07 8.5 rpy=0 90 0 -> (none)
- joint Bed_joint: origin xyz=14.959 1.57 -21.18 rpy=0 270 4.829673E-06 -> (none)
- joint BigDrawer_joint: origin xyz=4.690001 0.4299984 -20.76 rpy=0 90 -4.829673E-06 -> (none)
- joint Book.1_joint: origin xyz=15.493 4.364998 -27.998 rpy=-6.830189E-06 0 0 -> (none)
- joint Book.2_joint: origin xyz=15.695 4.445 -27.99 rpy=-6.830189E-06 0 0 -> (none)
- joint Book.3_joint: origin xyz=15.94 4.376997 -28.055 rpy=-6.830189E-06 0 0 -> (none)
- joint Book.4_joint: origin xyz=16.167 4.294998 -28.096 rpy=-6.830189E-06 0 0 -> (none)
- joint Book.5_joint: origin xyz=16.596 4.118 -28.093 rpy=-4.829673E-06 0 90 -> (none)
- joint Bookshelf_1_joint: origin xyz=16.07 2.529997 -27.99 rpy=-6.830189E-06 0 0 -> (none)
- joint Bookshelf_2_joint: origin xyz=-17.705 4.031 8.915998 rpy=0 90 0 -> (none)
- joint Bookshelf_joint: origin xyz=15.94 3.93 -27.99001 rpy=-6.830189E-06 0 0 -> (none)
- joint BoxshelfModel_joint: origin xyz=-0.5699978 1.145 10.17 rpy=0 180 0 -> (none)
- joint BroomBottom_joint: origin xyz=7.702 -0.23 9.919 rpy=288.4907 90 270 -> (none)
- joint BroomTop_joint: origin xyz=7.702 -0.23 9.919 rpy=288.4907 90 270 -> (none)
- joint Chair_1_joint: origin xyz=-11.28 0.806 -9.308001 rpy=0 90 0 -> (none)
- joint Chair_2_joint: origin xyz=-16.64 0.806 -6.28 rpy=0 270 0 -> (none)
- joint Chair_3_joint: origin xyz=-16.64 0.806 -9.308001 rpy=0 270 0 -> (none)
- joint Chair_joint: origin xyz=-11.28 0.806 -6.28 rpy=0 90 0 -> (none)
- joint Cube_10_joint: origin xyz=-7.849197 0.2898 10.139 rpy=0 90 0 -> (none)
- joint Cube_11_joint: origin xyz=-12.4913 1.986 10.1388 rpy=0 90 0 -> (none)
- joint Cube_12_joint: origin xyz=-10.981 0.5684 11.166 rpy=0 90 0 -> (none)
- joint Cube_13_joint: origin xyz=-7.810497 1.466 10.1388 rpy=0 90 0 -> (none)
- joint Cube_17042_joint: origin xyz=-13.39381 0.505 9.138998 rpy=0 180 0 -> (none)
- joint Cube_1_12959_joint: origin xyz=-7.131595 -0.8898 10.4106 rpy=0 180 0 -> (none)
- joint Cube_1_33376_joint: origin xyz=-18.274 -0.8744001 4.126998 rpy=0 90 0 -> (none)
- joint Cube_1_33534_joint: origin xyz=-7.131595 -0.3077999 10.4106 rpy=0 180 0 -> (none)
- joint Cube_1_66524_joint: origin xyz=-17.39 2.52 1.433998 rpy=-4.325711E-06 90.00001 0 -> (none)
- joint Cube_1_70777_joint: origin xyz=-7.131595 0.8602 10.4106 rpy=0 180 0 -> (none)
- joint Cube_1_86271_joint: origin xyz=-17.7031 1.5943 2.569999 rpy=0 180 0 -> (none)
- joint Cube_1_87286_joint: origin xyz=-7.131595 0.2772001 10.4106 rpy=0 180 0 -> (none)
- joint Cube_1_joint: origin xyz=-17.018 1.7092 -3.550002 rpy=0 90 0 -> (none)
- joint Cube_21715_joint: origin xyz=-11.016 0.1003999 9.139998 rpy=0 180 0 -> (none)
- joint Cube_21977_joint: origin xyz=5.2712 0.4545999 10.5104 rpy=90 4.829674E-06 0 -> (none)
- joint Cube_2_31866_joint: origin xyz=-17.703 1.5943 5.687999 rpy=0 180 0 -> (none)
- joint Cube_2_60947_joint: origin xyz=-7.803396 -0.6298 10.4106 rpy=0 180 0 -> (none)
- joint Cube_2_61029_joint: origin xyz=-7.803396 -0.0478 10.4106 rpy=0 180 0 -> (none)
- joint Cube_2_70115_joint: origin xyz=-7.803396 0.5372 10.4106 rpy=0 180 0 -> (none)
- joint Cube_2_70553_joint: origin xyz=-7.803396 1.1202 10.4106 rpy=0 180 0 -> (none)
- joint Cube_2_8193_joint: origin xyz=-17.39 2.0782 2.197699 rpy=-4.325711E-06 90.00001 0 -> (none)
- joint Cube_2_99358_joint: origin xyz=-18.274 0.1075 2.590997 rpy=0 90 0 -> (none)
- joint Cube_2_joint: origin xyz=-17.018 4.3293 -2.178802 rpy=0 90 0 -> (none)
- joint Cube_33884_joint: origin xyz=-8.610298 0.24633 9.129999 rpy=0 180 0 -> (none)
- joint Cube_34343_joint: origin xyz=-7.131595 -0.04500002 9.117199 rpy=0 180 0 -> (none)
- joint Cube_34559_joint: origin xyz=-15.8823 3.5486 -2.152702 rpy=0 90 0 -> (none)
- joint Cube_3736_joint: origin xyz=-14.91801 0.501 9.130997 rpy=0 0 0 -> (none)
- joint Cube_3_28928_joint: origin xyz=-17.923 1.3083 4.128599 rpy=0 90 0 -> (none)
- joint Cube_3_59990_joint: origin xyz=-6.469993 1.1202 10.411 rpy=0 180 0 -> (none)
- joint Cube_3_62137_joint: origin xyz=-17.39 2.968 2.197999 rpy=-4.325711E-06 90.00001 0 -> (none)
- joint Cube_3_73054_joint: origin xyz=-6.469993 -0.0478 10.411 rpy=0 180 0 -> (none)
- joint Cube_3_76169_joint: origin xyz=-18.274 0.1075 5.663 rpy=0 90 0 -> (none)
- joint Cube_3_83299_joint: origin xyz=-6.469993 -0.6298 10.411 rpy=0 180 0 -> (none)
- joint Cube_3_92970_joint: origin xyz=-6.469993 0.5372 10.411 rpy=0 180 0 -> (none)
- joint Cube_3_joint: origin xyz=-17.018 2.7033 -2.178804 rpy=0 90 0 -> (none)
- joint Cube_44086_joint: origin xyz=-16.0527 0.1074 4.126798 rpy=0 90 0 -> (none)
- joint Cube_4_14793_joint: origin xyz=-17.9106 2.5267 2.197999 rpy=-4.325711E-06 90.00001 0 -> (none)
- joint Cube_4_49644_joint: origin xyz=-10.9812 -0.862 10.1388 rpy=0 90 0 -> (none)
- joint Cube_4_56488_joint: origin xyz=-18.274 -0.8744001 7.302999 rpy=0 90 0 -> (none)
- joint Cube_4_65253_joint: origin xyz=-17.4512 1.194 4.155298 rpy=0 90 0 -> (none)
- joint Cube_4_joint: origin xyz=-17.01801 -0.832 -2.178806 rpy=0 90 0 -> (none)
- joint Cube_59574_joint: origin xyz=-16.7794 2.5219 2.187299 rpy=0 90 0 -> (none)
- joint Cube_5_74574_joint: origin xyz=-15.61611 0.5071 10.1388 rpy=0 90 0 -> (none)
- joint Cube_5_89013_joint: origin xyz=-17.4512 0.5015 5.768798 rpy=0 90 0 -> (none)
- joint Cube_5_joint: origin xyz=-17.9742 1.7165 -2.178802 rpy=0 90 0 -> (none)
- joint Cube_60132_joint: origin xyz=-16.067 0.5042 8.056999 rpy=0 90 0 -> (none)
- joint Cube_62369_joint: origin xyz=-7.131595 0.54 9.117199 rpy=0 180 0 -> (none)
- joint Cube_68380_joint: origin xyz=-15.5959 1.5943 4.128599 rpy=0 90 0 -> (none)
- joint Cube_6_41405_joint: origin xyz=-17.4512 1.9925 7.261599 rpy=0 90 0 -> (none)
- joint Cube_6_77647_joint: origin xyz=-14.17001 0.5071 10.139 rpy=0 90 0 -> (none)
- joint Cube_6_joint: origin xyz=-17.018 1.39 -2.178804 rpy=0 90 0 -> (none)
- joint Cube_75106_joint: origin xyz=-7.927597 1.6718 9.113199 rpy=0 180 0 -> (none)
- joint Cube_76983_joint: origin xyz=-17.3896 2.5202 2.944999 rpy=-4.325711E-06 90.00001 0 -> (none)
- joint Cube_7_63222_joint: origin xyz=-12.6616 0.5071 10.139 rpy=0 90 0 -> (none)
- joint Cube_7_79703_joint: origin xyz=-17.451 0.5015 7.292499 rpy=0 90 0 -> (none)
- joint Cube_7_joint: origin xyz=-17.018 0.1500001 -2.178804 rpy=0 90 0 -> (none)
- joint Cube_81478_joint: origin xyz=-7.131595 1.123 9.117199 rpy=0 180 0 -> (none)
- joint Cube_84650_joint: origin xyz=-7.131996 -0.627 9.110999 rpy=0 180 0 -> (none)
- joint Cube_87951_joint: origin xyz=-16.0626 0.5042 6.528999 rpy=0 90 0 -> (none)
- joint Cube_8_joint: origin xyz=-9.369199 0.5071 10.139 rpy=0 90 0 -> (none)
- joint Cube_97832_joint: origin xyz=-15.8932 0.9043 -2.183702 rpy=0 90 0 -> (none)
- joint Cube_9_joint: origin xyz=-6.354995 0.5071 10.14 rpy=0 90 0 -> (none)
- joint Cube_joint: origin xyz=-17.0177 1.7092 -0.8097024 rpy=0 90 0 -> (none)
- joint Door_02_1_joint: origin xyz=3.702 -1.045 -11.03 rpy=0 343.9 0 -> (none)
- joint Door_02_joint: origin xyz=3.702 -1.045 3.05 rpy=0 34.99999 0 -> (none)
- joint Drawer_1_joint: origin xyz=4.68 0.07999611 -24.74 rpy=0 90 -4.829673E-06 -> (none)
- joint Drawer_2_joint: origin xyz=17.739 0.07999992 -25.5 rpy=0 270 4.829673E-06 -> (none)
- joint Drawer_joint: origin xyz=17.739 0.07999802 -16.83 rpy=0 270 4.829673E-06 -> (none)
- joint Floor_Carpet_Grey_joint: origin xyz=3.577 -0.91956 11.534 rpy=0 0 0 -> (none)
- joint Floor_Carpet_Tiles_1_joint: origin xyz=-17.37 -0.919 3.899999 rpy=0 0 0 -> (none)
- joint Floor_Carpet_Tiles_2_joint: origin xyz=-17.37 -0.919 8.9 rpy=0 0 0 -> (none)
- joint Floor_Carpet_Tiles_3_joint: origin xyz=-13.44 -0.919 -1.1 rpy=0 0 0 -> (none)
- joint Floor_Carpet_Tiles_4_joint: origin xyz=-13.44 -0.919 3.9 rpy=0 0 0 -> (none)
- joint Floor_Carpet_Tiles_5_joint: origin xyz=-13.44001 -0.919 8.900002 rpy=0 0 0 -> (none)
- joint Floor_Carpet_Tiles_6_joint: origin xyz=-8.440003 -0.919 -1.100001 rpy=0 0 0 -> (none)
- joint Floor_Carpet_Tiles_7_joint: origin xyz=-8.440003 -0.919 3.899999 rpy=0 0 0 -> (none)
- joint Floor_Carpet_Tiles_8_joint: origin xyz=-8.440004 -0.919 8.900002 rpy=0 0 0 -> (none)
- joint Floor_Carpet_Tiles_joint: origin xyz=-17.37 -0.919 -1.100002 rpy=0 0 0 -> (none)
- joint Floor_Vinyl_joint: origin xyz=11.432 -0.91956 5.102 rpy=0 270 0 -> (none)
- joint Floor_Wood_10_joint: origin xyz=16.06 -0.9190006 -21.56002 rpy=0 0 0 -> (none)
- joint Floor_Wood_11_joint: origin xyz=16.06 -0.9190044 -26.56002 rpy=0 0 0 -> (none)
- joint Floor_Wood_1_joint: origin xyz=6.059996 -0.9189987 -16.55999 rpy=0 0 0 -> (none)
- joint Floor_Wood_2_joint: origin xyz=6.060001 -0.9190006 -21.56 rpy=0 0 0 -> (none)
- joint Floor_Wood_3_joint: origin xyz=6.060007 -0.9190006 -26.56001 rpy=0 0 0 -> (none)
- joint Floor_Wood_4_joint: origin xyz=11.06 -0.9190025 -11.55999 rpy=0 0 0 -> (none)
- joint Floor_Wood_5_joint: origin xyz=11.06 -0.9189987 -16.55999 rpy=0 0 0 -> (none)
- joint Floor_Wood_6_joint: origin xyz=11.06 -0.9190006 -21.56001 rpy=0 0 0 -> (none)
- joint Floor_Wood_7_joint: origin xyz=11.06 -0.9190044 -26.56002 rpy=0 0 0 -> (none)
- joint Floor_Wood_8_joint: origin xyz=16.06 -0.9190025 -11.55999 rpy=0 0 0 -> (none)
- joint Floor_Wood_9_joint: origin xyz=16.06 -0.9189987 -16.56 rpy=0 0 0 -> (none)
- joint Floor_Wood_joint: origin xyz=6.059988 -0.9190025 -11.55998 rpy=0 0 0 -> (none)
- joint Items_CrowBar_01_joint: origin xyz=3.115 -0.233 -2.41 rpy=0 0 0 -> (none)
- joint Items_Drill_01_joint: origin xyz=3.233 1.195 -2.635 rpy=0 0 0 -> (none)
- joint Items_FlashLight_01_joint: origin xyz=3.027 2.113 -4.699 rpy=90 0 0 -> (none)
- joint Items_FryPan_01_joint: origin xyz=-16.577 0.747 1.762 rpy=0 240.0001 0 -> (none)
- joint Items_Hammer_01_joint: origin xyz=3.12 0.917 -2.16 rpy=0 0 180 -> (none)
- joint Items_ScrewDriver_01_joint: origin xyz=3.205001 2.425 -1.852913 rpy=270 0.0001678311 0 -> (none)
- joint Items_ScrewDriver_02_joint: origin xyz=3.205 2.426 -2.158 rpy=270 0.0001678311 0 -> (none)
- joint Items_ScrewDriver_03_joint: origin xyz=3.204999 2.426 -2.432045 rpy=270 0.0001678311 0 -> (none)
- joint Items_SledgeHammer_01_joint: origin xyz=3.218 -0.141 -7.317 rpy=90 270 0 -> (none)
- joint Items_SmartPhone_01_joint: origin xyz=-11.626 1.673 -12.796 rpy=0 13.05 0 -> (none)
- joint Items_Spanner_01_joint: origin xyz=3.122 2.068 -2.697 rpy=0 345 0 -> (none)
- joint Items_Wrench_01_joint: origin xyz=3.014 -0.476 -5.38 rpy=0 180 0 -> (none)
- joint Lamp_joint: origin xyz=17.739 1.939999 -16.83 rpy=-6.830189E-06 0 0 -> (none)
- joint MicrowaveBack_joint: origin xyz=-17.29 2.52 2.189999 rpy=-4.325711E-06 90.00001 0 -> (none)
- joint MicrowaveFrontModel_joint: origin xyz=-17.29 2.52 2.189998 rpy=-4.325711E-06 90.00001 0 -> (none)
- joint Mirror.1_joint: origin xyz=4.370001 1.129965 -27.17002 rpy=0 90 -4.829673E-06 -> (none)
- joint Mirror_joint: origin xyz=13.4 4.48 11.104 rpy=0 180 0 -> (none)
- joint Plunger_joint: origin xyz=8.93 2.188002 10.57 rpy=349.6 0 0 -> (none)
- joint Prop_Bar_Bench_joint: origin xyz=-14.37 -0.919 -12.77 rpy=0 180 0 -> (none)
- joint Prop_BathMat_Blue_joint: origin xyz=15.955 -0.911 8.335 rpy=0 0 0 -> (none)
- joint Prop_Big_Clock_joint: origin xyz=2.39 -0.919 -24.21 rpy=0 270 0 -> (none)
- joint Prop_Bonzai_joint: origin xyz=-17.714 2.42 -23.86 rpy=0 90 0 -> (none)
- joint Prop_Cupboard_03_joint: origin xyz=-17.51 -0.919 -23.893 rpy=0 90 0 -> (none)
- joint Prop_Curtains_Blue_1_joint: origin xyz=-12.51 -3.415 -28.52 rpy=0 0 0 -> (none)
- joint Prop_Curtains_Blue_2_joint: origin xyz=-18.17 -3.415 -17.66 rpy=0 90 0 -> (none)
- joint Prop_Curtains_Blue_3_joint: origin xyz=-18.17 -3.415 -7.8 rpy=0 90 0 -> (none)
- joint Prop_Curtains_Blue_joint: origin xyz=-2.48 -3.415 -28.52 rpy=0 0 0 -> (none)
- joint Prop_Curtains_Red_1_joint: origin xyz=18.78 5.799974 -20.82001 rpy=-1.207425E-05 270.0002 4.105219E-05 -> (none)
- joint Prop_Curtains_Red_joint: origin xyz=9.639999 4.589972 -28.52002 rpy=0 0 0 -> (none)
- joint Prop_Fireplace_02_joint: origin xyz=2.52 -0.95 -20.61 rpy=0 270 0 -> (none)
- joint Prop_Plant_02_joint: origin xyz=-10.58 1.634 -12.7 rpy=0 0 0 -> (none)
- joint Prop_Plant_joint: origin xyz=3.065 4.08 8.524 rpy=0 0 0 -> (none)
- joint Prop_Rug_03_joint: origin xyz=-7.422 -0.99 -27.518 rpy=0 0 0 -> (none)
- joint Prop_Shelf_011_2_joint: origin xyz=3.16 -0.919 -8.66 rpy=0 270 0 -> (none)
- joint Prop_Shelf_011_joint: origin xyz=3.16 -0.919 -2.4 rpy=0 270 0 -> (none)
- joint Prop_Shelf_04_joint: origin xyz=3.060003 -0.919 -5.55 rpy=0 270 0 -> (none)
- joint Prop_Speaker_02_1_joint: origin xyz=2.58 -0.919 -27.5 rpy=0 315 0 -> (none)
- joint Prop_Speaker_02_joint: origin xyz=-17.14 -0.919 -27.5 rpy=0 45 0 -> (none)
- joint Prop_ToiletSeat_01_joint: origin xyz=10.42186 0.6673605 10.48428 rpy=0 180 0 -> (none)
- joint Prop_Toilet_01_joint: origin xyz=10.415 -0.911 11.267 rpy=0 180 0 -> (none)
- joint Prop_WallArt_01_joint: origin xyz=3.406 3.93 -20.639 rpy=0 270 0 -> (none)
- joint Prop_WallArt_02_joint: origin xyz=3.406 3.5 -22.302 rpy=0 270 0 -> (none)
- joint Prop_WallArt_03_joint: origin xyz=3.406 4.32 -18.934 rpy=0 270 0 -> (none)
- joint Prop_shelf_01_1_joint: origin xyz=3.060003 3.35026 -5.55 rpy=0 270 0 -> (none)
- joint Prop_shelf_01_joint: origin xyz=3.057002 3.35026 7.36 rpy=0 270 0 -> (none)
- joint Refridgerator_Door_joint: origin xyz=-16.94 1.72 -2.190004 rpy=0 90 0 -> (none)
- joint Refridgerator_Empty_joint: origin xyz=-16.94 1.72 -2.190002 rpy=0 90 0 -> (none)
- joint Refridgerator_UpperDrawer_joint: origin xyz=-16.94 1.72 -2.190004 rpy=0 90 0 -> (none)
- joint SI_Env_Wall_01_10_joint: origin xyz=-18.31 -0.573 11.19 rpy=0 180 0 -> (none)
- joint SI_Env_Wall_01_11_joint: origin xyz=-18.3 -0.573 -3.9779 rpy=0 90 0 -> (none)
- joint SI_Env_Wall_01_12_joint: origin xyz=-18.3 -0.573 -14.118 rpy=0 90 0 -> (none)
- joint SI_Env_Wall_01_13_joint: origin xyz=-18.3 -0.573 -28.715 rpy=0 90 0 -> (none)
- joint SI_Env_Wall_01_14_joint: origin xyz=-18.284 -3.714 -21.787 rpy=0 90 0 -> (none)
- joint SI_Env_Wall_01_15_joint: origin xyz=-18.284 -3.714 -11.9077 rpy=0 90 0 -> (none)
- joint SI_Env_Wall_01_16_joint: origin xyz=-18.26 11.427 -28.58 rpy=0 0 180 -> (none)
- joint SI_Env_Wall_01_17_joint: origin xyz=-8.7521 11.427 -28.58 rpy=0 0 180 -> (none)
- joint SI_Env_Wall_01_18_joint: origin xyz=1.102 11.427 -28.58 rpy=0 0 180 -> (none)
- joint SI_Env_Wall_01_19_joint: origin xyz=-15.7779 -0.573 -28.58 rpy=0 0 0 -> (none)
- joint SI_Env_Wall_01_1_joint: origin xyz=3.444 -0.573 -2.16 rpy=0 270 0 -> (none)
- joint SI_Env_Wall_01_20_joint: origin xyz=-6.27 -0.573 -28.58 rpy=0 0 0 -> (none)
- joint SI_Env_Wall_01_21_joint: origin xyz=5.9476 -0.573 -28.58 rpy=0 0 0 -> (none)
- joint SI_Env_Wall_01_22_joint: origin xyz=-8.6709 -3.69 -28.58 rpy=0 0 0 -> (none)
- joint SI_Env_Wall_01_23_joint: origin xyz=1.181 -3.69 -28.58 rpy=0 0 0 -> (none)
- joint SI_Env_Wall_01_24_joint: origin xyz=13.481 -3.69 -28.58 rpy=0 0 0 -> (none)
- joint SI_Env_Wall_01_25_joint: origin xyz=13.396 11.427 -28.58 rpy=0 0 180 -> (none)
- joint SI_Env_Wall_01_26_joint: origin xyz=18.794 -0.573 -28.58 rpy=0 0 0 -> (none)
- joint SI_Env_Wall_01_27_joint: origin xyz=18.73 -2.56 -16.074 rpy=0 270.0002 0 -> (none)
- joint SI_Env_Wall_01_28_joint: origin xyz=18.70999 11.427 -30.908 rpy=0 270.0002 180 -> (none)
- joint SI_Env_Wall_01_29_joint: origin xyz=18.71 -0.573 -25.4816 rpy=0 270.0002 0 -> (none)
- joint SI_Env_Wall_01_2_joint: origin xyz=3.444 -0.573 -16.26 rpy=0 270 0 -> (none)
- joint SI_Env_Wall_01_30_joint: origin xyz=18.70999 11.427 -16.178 rpy=0 270.0002 180 -> (none)
- joint SI_Env_Wall_01_31_joint: origin xyz=18.71 -0.573 -1.0812 rpy=0 270.0002 0 -> (none)
- joint SI_Env_Wall_01_32_joint: origin xyz=18.72 11.427 -10.23 rpy=0 180.0003 180 -> (none)
- joint SI_Env_Wall_01_33_joint: origin xyz=3.4992 -0.573 -10.23 rpy=0 180.0003 0 -> (none)
- joint SI_Env_Wall_01_34_joint: origin xyz=3.5201 11.427 -10.1001 rpy=0 90.0005 180 -> (none)
- joint SI_Env_Wall_01_35_joint: origin xyz=3.52 -0.573 -28.613 rpy=0 90.0005 0 -> (none)
- joint SI_Env_Wall_01_3_joint: origin xyz=-6.1679 -0.573 11.19 rpy=0 180 0 -> (none)
- joint SI_Env_Wall_01_4_joint: origin xyz=3.444 11.427 -28.6875 rpy=0 270 180 -> (none)
- joint SI_Env_Wall_01_5_joint: origin xyz=3.448 11.427 11.19 rpy=0 180 180 -> (none)
- joint SI_Env_Wall_01_6_joint: origin xyz=-16.127 11.427 11.19 rpy=0 180 180 -> (none)
- joint SI_Env_Wall_01_7_joint: origin xyz=-18.3 11.427 11.19 rpy=0 90 180 -> (none)
- joint SI_Env_Wall_01_8_joint: origin xyz=-18.3 11.427 -21.4041 rpy=0 90 180 -> (none)
- joint SI_Env_Wall_01_9_joint: origin xyz=-18.3 11.427 -11.3813 rpy=0 90 180 -> (none)
- joint SI_Env_Wall_01_joint: origin xyz=3.444 -0.573 11.732 rpy=0 270 0 -> (none)
- joint SI_Env_Wall_CornerBlock_large_10_joint: origin xyz=18.74 11.42 -16.061 rpy=0 270.0002 90 -> (none)
- joint SI_Env_Wall_CornerBlock_large_11_joint: origin xyz=18.74 -0.612 -16.026 rpy=0 270.0002 90 -> (none)
- joint SI_Env_Wall_CornerBlock_large_1_joint: origin xyz=-18.31 11.4261 -21.739 rpy=0 90 90 -> (none)
- joint SI_Env_Wall_CornerBlock_large_2_joint: origin xyz=-18.31 -0.6823 -21.739 rpy=0 90 90 -> (none)
- joint SI_Env_Wall_CornerBlock_large_3_joint: origin xyz=1.17 11.42 -28.59 rpy=0 0 90 -> (none)
- joint SI_Env_Wall_CornerBlock_large_4_joint: origin xyz=1.22 -0.6124 -28.59 rpy=0 0 90 -> (none)
- joint SI_Env_Wall_CornerBlock_large_5_joint: origin xyz=-6.1333 0.6365 11.1834 rpy=0 0 90 -> (none)
- joint SI_Env_Wall_CornerBlock_large_6_joint: origin xyz=-16.1421 5.4293 11.1834 rpy=0 0 90 -> (none)
- joint SI_Env_Wall_CornerBlock_large_7_joint: origin xyz=-3.972 5.4293 11.1834 rpy=0 0 90 -> (none)
- joint SI_Env_Wall_CornerBlock_large_8_joint: origin xyz=13.492 11.42 -28.59 rpy=0 0 90 -> (none)
- joint SI_Env_Wall_CornerBlock_large_9_joint: origin xyz=13.52 -0.612 -28.59 rpy=0 0 90 -> (none)
- joint SI_Env_Wall_CornerBlock_large_joint: origin xyz=-5.347 11.4 11.1834 rpy=0 0 90 -> (none)
- joint SI_Env_Wall_Door_Small_01_1_joint: origin xyz=3.444 -0.573 -8.77 rpy=0 270 0 -> (none)
- joint SI_Env_Wall_Door_Small_01_2_joint: origin xyz=3.52 -0.573 -16.27 rpy=0 90.00011 0 -> (none)
- joint SI_Env_Wall_Door_Small_01_joint: origin xyz=3.444 -0.573 5.32 rpy=0 270 0 -> (none)
- joint SI_Env_Wall_Large_Window_05_1_joint: origin xyz=-18.3 2.47 -11.41 rpy=0 90 0 -> (none)
- joint SI_Env_Wall_Large_Window_05_2_joint: origin xyz=-18.3 2.47 -21.42 rpy=0 90 0 -> (none)
- joint SI_Env_Wall_Large_Window_05_3_joint: origin xyz=-8.72 2.47 -28.58 rpy=0 0 0 -> (none)
- joint SI_Env_Wall_Large_Window_05_4_joint: origin xyz=1.11 2.47 -28.58 rpy=0 0 0 -> (none)
- joint SI_Env_Wall_Large_Window_05_5_joint: origin xyz=13.41 2.47 -28.58 rpy=0 0 0 -> (none)
- joint SI_Env_Wall_Large_Window_05_6_joint: origin xyz=18.73 3.6 -16.163 rpy=0 270.0002 0 -> (none)
- joint SI_Env_Wall_Large_Window_05_joint: origin xyz=-16.1438 2.47 11.19 rpy=0 180 0 -> (none)
- joint SI_Food_Meat_Steak_Raw_joint: origin xyz=-16.964 2.917 -2.189 rpy=0 0 0 -> (none)
- joint SM_Bowl_1_joint: origin xyz=0.5294275 3.315002 9.759998 rpy=270 0 0 -> (none)
- joint SM_Bowl_2_joint: origin xyz=-2.850574 2.816498 9.759998 rpy=270 0 0 -> (none)
- joint SM_Bowl_3_joint: origin xyz=-2.850574 3.315002 9.759998 rpy=270 0 0 -> (none)
- joint SM_Bowl_Small_1_joint: origin xyz=-1.385574 4.880005 9.640499 rpy=270 0 0 -> (none)
- joint SM_Bowl_Small_2_joint: origin xyz=-0.7055731 4.405502 9.6405 rpy=270 0 0 -> (none)
- joint SM_Bowl_Small_3_joint: origin xyz=-0.7055731 4.880005 9.6405 rpy=270 0 0 -> (none)
- joint SM_Bowl_Small_joint: origin xyz=-1.385574 4.405502 9.640499 rpy=270 0 0 -> (none)
- joint SM_Bowl_joint: origin xyz=0.5294275 2.816498 9.759998 rpy=270 0 0 -> (none)
- joint SM_Fork_Dinner_15572_joint: origin xyz=-16.295 1.463 4.655999 rpy=270 0 0 -> (none)
- joint SM_Fork_Dinner_17398_joint: origin xyz=-16.295 1.463 4.226998 rpy=270 0 0 -> (none)
- joint SM_Fork_Dinner_69885_joint: origin xyz=-16.295 1.463 4.457999 rpy=270 0 0 -> (none)
- joint SM_Fork_Dinner_joint: origin xyz=-16.295 1.463 4.838998 rpy=270 0 0 -> (none)
- joint SM_Knife_Table_12175_joint: origin xyz=-16.343 1.441 5.391999 rpy=90 0 0 -> (none)
- joint SM_Knife_Table_48929_joint: origin xyz=-16.343 1.441 5.230999 rpy=90 0 0 -> (none)
- joint SM_Knife_Table_84538_joint: origin xyz=-16.343 1.441 5.568999 rpy=90 0 0 -> (none)
- joint SM_Knife_Table_joint: origin xyz=-16.343 1.441 5.063999 rpy=90 0 0 -> (none)
- joint SM_Plate_Classic_16cm_1_joint: origin xyz=-1.125576 3.070007 9.749996 rpy=270 0 0 -> (none)
- joint SM_Plate_Classic_16cm_2_joint: origin xyz=-1.125576 3.285004 9.749996 rpy=270 0 0 -> (none)
- joint SM_Plate_Classic_16cm_3_joint: origin xyz=-1.125576 3.535004 9.749996 rpy=270 0 0 -> (none)
- joint SM_Plate_Classic_16cm_joint: origin xyz=-1.125576 2.839996 9.749996 rpy=270 0 0 -> (none)
- joint SM_Plate_Classic_21cm_1_joint: origin xyz=-1.125576 1.544998 9.605 rpy=270 0 0 -> (none)
- joint SM_Plate_Classic_21cm_2_joint: origin xyz=-1.125576 1.789993 9.605 rpy=270 0 0 -> (none)
- joint SM_Plate_Classic_21cm_3_joint: origin xyz=-1.125576 2.080002 9.605 rpy=270 0 0 -> (none)
- joint SM_Plate_Classic_21cm_joint: origin xyz=-1.125576 1.229996 9.605 rpy=270 0 0 -> (none)
- joint SM_Plate_Classic_26cm_1_joint: origin xyz=-2.668575 1.315002 9.868156 rpy=270 0 0 -> (none)
- joint SM_Plate_Classic_26cm_2_joint: origin xyz=-2.668575 1.639999 9.868156 rpy=270 0 0 -> (none)
- joint SM_Plate_Classic_26cm_3_joint: origin xyz=-2.668575 1.914993 9.868156 rpy=270 0 0 -> (none)
- joint SM_Plate_Classic_26cm_joint: origin xyz=-2.668575 1.020004 9.868156 rpy=270 0 0 -> (none)
- joint SM_Saucer_1_joint: origin xyz=-2.66 -0.1549988 9.659996 rpy=270 0 0 -> (none)
- joint SM_Saucer_2_joint: origin xyz=-2.66 0.1450043 9.659996 rpy=270 0 0 -> (none)
- joint SM_Saucer_3_joint: origin xyz=-2.66 0.3450012 9.659996 rpy=270 0 0 -> (none)
- joint SM_Saucer_joint: origin xyz=-2.66 -0.3950043 9.659996 rpy=270 0 0 -> (none)
- joint SM_Spoon_Soup_10143_joint: origin xyz=-16.315 1.432 3.328998 rpy=270 0 0 -> (none)
- joint SM_Spoon_Soup_24722_joint: origin xyz=-16.315 1.432 3.561997 rpy=270 0 0 -> (none)
- joint SM_Spoon_Soup_88278_joint: origin xyz=-16.315 1.432 3.070998 rpy=270 0 0 -> (none)
- joint SM_Spoon_Soup_joint: origin xyz=-16.315 1.432 2.824997 rpy=270 0 0 -> (none)
- joint SM_TraySet_Mid_joint: origin xyz=-1.002998 6.078 9.972 rpy=270 0 0 -> (none)
- joint SO_Boxfile_01_joint: origin xyz=3.1663 2.045 -8.281821 rpy=0 270.0002 0 -> (none)
- joint SO_Boxfile_03_joint: origin xyz=3.1494 2.045 -8.480217 rpy=0 270.0002 0 -> (none)
- joint SO_Boxfile_05_joint: origin xyz=3.14 2.045 -8.725733 rpy=0 270.0002 0 -> (none)
- joint SO_Boxfile_06_joint: origin xyz=3.135 2.045 -8.952489 rpy=0 270.0002 0 -> (none)
- joint SO_Broom_joint: origin xyz=2.884468 -0.894 -3.863593 rpy=0 0 354.2464 -> (none)
- joint SO_CarboardBox_01_joint: origin xyz=3.084 4.087 -6.447 rpy=0 0 0 -> (none)
- joint SO_Clipboard_joint: origin xyz=-18.46 6.8 4.09 rpy=90 90 0 -> (none)
- joint SO_Papers_03_joint: origin xyz=3.126 0.855 -8.923 rpy=0 0 0 -> (none)
- joint SO_Pen_01_joint: origin xyz=3.129592 0.888 -8.303489 rpy=0 330.0001 0 -> (none)
- joint SO_Pen_02_joint: origin xyz=3.055438 0.8880001 -8.365969 rpy=0 330.0001 0 -> (none)
- joint SO_Pinboard_01_joint: origin xyz=3.389 2.333 7.341 rpy=0 269.9999 0 -> (none)
- joint SO_Plant_01_joint: origin xyz=-17.36 1.64 -12.64 rpy=0 0 0 -> (none)
- joint SO_Plant_02_joint: origin xyz=-17.8 4.110114 8.835001 rpy=0 90 0 -> (none)
- joint SO_Plant_03_joint: origin xyz=17.41157 4.035475 -27.85461 rpy=0 0 0 -> (none)
- joint SO_RubixCube_joint: origin xyz=3.023 1.677 -6.291 rpy=0 0 0 -> (none)
- joint SO_Rug_01_joint: origin xyz=11.038 -0.9190006 -21.173 rpy=0 90 0 -> (none)
- joint Sink.2_joint: origin xyz=-16.839 0.56 9.922998 rpy=0 90 0 -> (none)
- joint Sink1_DoorL_joint: origin xyz=-11.01 0.56 10.1 rpy=0 180 0 -> (none)
- joint Sink1_DoorR_joint: origin xyz=-11.01 0.56 10.1 rpy=0 180 0 -> (none)
- joint Sink1_Drawer2_joint: origin xyz=-11.01 0.56 10.1 rpy=0 180 0 -> (none)
- joint Sink1_Drawer3_joint: origin xyz=-11.01 0.56 10.1 rpy=0 180 0 -> (none)
- joint Sink1_Drawer4_joint: origin xyz=-11.01 0.56 10.1 rpy=0 180 0 -> (none)
- joint Sink1_Drawer5_joint: origin xyz=-11.01 0.56 10.1 rpy=0 180 0 -> (none)
- joint Sink1_Empty_joint: origin xyz=-11.01 0.56 10.1 rpy=0 180 0 -> (none)
- joint Sink1_OvenDoor_joint: origin xyz=-11.01 0.5599999 10.1 rpy=0 180 0 -> (none)
- joint Sink1_SinkDoor_joint: origin xyz=-11.01 0.29063 10.1 rpy=0 180 0 -> (none)
- joint Sink_DoorL_joint: origin xyz=-17.01 0.56 4.129998 rpy=0 90 0 -> (none)
- joint Sink_DoorR_joint: origin xyz=-17.01 0.56 4.129997 rpy=0 90 0 -> (none)
- joint Sink_Drawer1_joint: origin xyz=-16.597 0.56 4.129999 rpy=0 90 0 -> (none)
- joint Sink_Drawer2_joint: origin xyz=-17.01 0.56 4.129999 rpy=0 90 0 -> (none)
- joint Sink_WithoutDrawers_joint: origin xyz=-17.01 0.56 4.129999 rpy=0 90 0 -> (none)
- joint Sofa.1_joint: origin xyz=-7.56 0.28 -14.73 rpy=0 180 0 -> (none)
- joint TVTable_joint: origin xyz=-7.552001 0.34 -27.778 rpy=0 180 0 -> (none)
- joint TV_joint: origin xyz=-7.442001 2 -27.728 rpy=0 0 0 -> (none)
- joint Table_joint: origin xyz=-13.58 1.249 -7.778 rpy=0 90 0 -> (none)
- joint TallLamp_joint: origin xyz=4.789999 2.199999 -17.32 rpy=-6.830189E-06 0 0 -> (none)
- joint Toilet_Paper_joint: origin xyz=11.885 0.445 10.832 rpy=0 180 0 -> (none)
- joint Towel_Rack_joint: origin xyz=18.52802 1.824098 2.742241 rpy=0 270 0 -> (none)
- joint Trashcan1Cap_joint: origin xyz=-5.0555 1.5265 9.9825 rpy=270 0 0 -> (none)
- joint Trashcan1_joint: origin xyz=-5.052871 -0.866 9.978473 rpy=270 0 0 -> (none)
- joint Upper_joint: origin xyz=-1.544999 3.855499 10.17 rpy=0 180 180 -> (none)
- joint Wall_01_Blue_1_joint: origin xyz=19.055 -0.692461 11.321 rpy=0 270 0 -> (none)
- joint Wall_01_Blue_2_joint: origin xyz=19.055 11.43 -1.2792 rpy=0 270 179.9997 -> (none)
- joint Wall_01_Blue_3_joint: origin xyz=3.4759 -0.692461 11.2 rpy=0 180.0002 0 -> (none)
- joint Wall_01_Blue_4_joint: origin xyz=19.0838 11.43 11.19998 rpy=8.837917E-12 180.0002 179.9997 -> (none)
- joint Wall_01_Blue_5_joint: origin xyz=3.525944 -0.692461 3.596399 rpy=0 90.00033 0 -> (none)
- joint Wall_01_Blue_6_joint: origin xyz=3.526 11.4293 11.248 rpy=-5.211021E-11 90.00033 179.9997 -> (none)
- joint Wall_01_Blue_7_joint: origin xyz=19.0899 -0.692461 -1.04 rpy=0 0.0004934811 0 -> (none)
- joint Wall_01_Blue_8_joint: origin xyz=3.5217 11.43 -1.039911 rpy=-1.08926E-11 0.0004934811 179.9997 -> (none)
- joint Wall_01_Blue_joint: origin xyz=19.055 -0.692461 3.6267 rpy=0 270 0 -> (none)
- joint Wall_Door_01_Blue_1_joint: origin xyz=3.521 -0.5679 -2.1477 rpy=0 90 0 -> (none)
- joint Wall_Window_01_Blue_joint: origin xyz=19.055 -0.692461 8.61 rpy=0 270 0 -> (none)
- joint appleGreen_1_joint: origin xyz=-17.665 2.456 4.159999 rpy=270 0 0 -> (none)
- joint appleGreen_joint: origin xyz=-17.335 2.456 3.513999 rpy=270 0 0 -> (none)
- joint appleRed_joint: origin xyz=-17.12 2.456 4.069999 rpy=270 0 0 -> (none)
- joint apricot_joint: origin xyz=-17.165 0.476 -2.348001 rpy=270.0198 0 0 -> (none)
- joint banana_joint: origin xyz=-17.828 2.896 -0.3220019 rpy=270 0 0 -> (none)
- joint bellPepperOrange_joint: origin xyz=-16.764 1.836 -2.884 rpy=270.0198 0 0 -> (none)
- joint bellPepperYellow_joint: origin xyz=-17.145 1.836 -2.796 rpy=270.0198 0 0 -> (none)
- joint bellpepperRed_joint: origin xyz=-16.974 1.836 -3.16 rpy=270.0198 0 0 -> (none)
- joint broccoli_joint: origin xyz=-16.449 0.642 -1.892001 rpy=0 0 0 -> (none)
- joint carrot_joint: origin xyz=-17.333 3.151 2.225998 rpy=-1.707547E-06 0 0 -> (none)
- joint cauliflower_joint: origin xyz=-16.354 0.42 -2.534 rpy=270.0198 0 0 -> (none)
- joint cherryRed_joint: origin xyz=-16.86 -0.661 -1.95 rpy=270.0198 0 0 -> (none)
- joint chiliPepper_joint: origin xyz=-16.638 -0.596 -1.701 rpy=0 0 0 -> (none)
- joint cucumber_joint: origin xyz=-16.655 1.809 -1.551002 rpy=270 0 0 -> (none)
- joint eggplant_joint: origin xyz=-16.492 1.733 -2.485 rpy=0 0 0 -> (none)
- joint fig_joint: origin xyz=-16.589 -0.596 -2.309 rpy=0 0 0 -> (none)
- joint garlic_joint: origin xyz=-16.735 -0.596 -2.646 rpy=270 0 0 -> (none)
- joint ground_joint: origin xyz=5.308927 2.7078 9.903153 rpy=0 0 0 -> (none)
- joint lemon_joint: origin xyz=-17.081 0.539 -3.014001 rpy=0 0 0 -> (none)
- joint lettuce_joint: origin xyz=-17.194 0.539 -1.816001 rpy=0 0 0 -> (none)
- joint oil_joint: origin xyz=-17.384 2.062249 -0.222 rpy=270 39.0218 0 -> (none)
- joint pawpaw_joint: origin xyz=-17.197 2.615 1.050998 rpy=270 0 0 -> (none)
- joint potatoYellow_1_joint: origin xyz=-16.461 2.337 10.235 rpy=270 0 0 -> (none)
- joint potatoYellow_joint: origin xyz=-16.662 2.337 10.023 rpy=270 0 0 -> (none)
- joint radish_1_joint: origin xyz=-17.271 2.87 9.940001 rpy=270 0 0 -> (none)
- joint radish_2_joint: origin xyz=-17.271 2.87 9.681 rpy=270 0 0 -> (none)
- joint radish_joint: origin xyz=-17.52 2.87 9.940001 rpy=270 0 0 -> (none)
- joint scp_mw_axe_joint: origin xyz=3.202 0.24 -6.187 rpy=345.0002 270 270 -> (none)
- joint scp_mw_baseball_bat_02_joint: origin xyz=3.257 3.364 -9.292 rpy=90 350.0104 0 -> (none)
- joint scp_mw_cleaver_knife_02_joint: origin xyz=-18.20407 3.65 8.952 rpy=0 0 180 -> (none)
- joint scp_mw_fire_poker_joint: origin xyz=3.139 -0.07 -17.599 rpy=2.347877E-05 269.9998 184.1453 -> (none)
- joint scp_mw_flyswatter_01_joint: origin xyz=3.163 -0.286 -8.394 rpy=270 0 0 -> (none)
- joint scp_mw_flyswatter_02_joint: origin xyz=3.023543 -0.3076015 -8.394 rpy=270 0 0 -> (none)
- joint scp_mw_kitchen_fork_joint: origin xyz=-18.25584 3.641 9.529 rpy=90 90 0 -> (none)
- joint scp_mw_kitchen_turner_joint: origin xyz=-18.19057 3.614 9.892 rpy=90 90 0 -> (none)
- joint scp_mw_knife_01_1_joint: origin xyz=-18.216 3.686 8.407 rpy=0 180 180 -> (none)
- joint scp_mw_knife_01_2_92314_joint: origin xyz=-17.627 2.183 8.666 rpy=3.585849E-05 105.2766 89.99985 -> (none)
- joint scp_mw_knife_01_2_joint: origin xyz=-18.216 3.723 8.699 rpy=0 180 180 -> (none)
- joint scp_mw_knife_01_joint: origin xyz=-18.216 3.638 8.068602 rpy=0 180 180 -> (none)
- joint scp_mw_rolling_pin_joint: origin xyz=-17.218 -0.445 1.368 rpy=90 0 0 -> (none)
- joint tomato_joint: origin xyz=-17.101 1.733 -2.17 rpy=270 0 0 -> (none)
- joint world_room_joint: origin xyz=0.0 0.03 0.0 rpy=0 0 0 -> (none)
